File: arduino/hardware/electronics/shield.sch (EAGLE design)
At the start: 22 parts

Commit message: Updated electronics
Parts:
- removed ESP8266-LEFT, ESP8266-RIGHT: (no value), pinhead:PINHD-1X8
- removed RELAY_1, RELAY_2: (no value), pinhead:PINHD-1X3
- added C1: 1uf, rcl:CPOL-EUTT2D5
- added CX1: 0.1uF, resistor:CXXC10B5
- added JP1: (no value), pinhead:PINHD-1X4
- added R8: 4.7k, eagle-ltspice:R0204/7
- added R9: S2220, varistor:S2220
- added S1: (no value), switch-dil:SD4-01
- added U$4: ESP8266_SHIELD, esp8266_shield:ESP8266_SHIELD
- IC1: value (none) -> 3.3V
Connections:
- removed net ESP8266_CH_PD: ESP8266-LEFT.3, R4.2
- removed net ESP_8266_TX: B1.15(RX3)
- removed net N$1: U$1.AC1, X1-1.KL, X2-1.KL, X3-1.KL
- new net DC+: S1.2, U$1.DC+
- new net GND4: B1.GND@4, DHT.2, LDR.2, TMP1.2, TMP2.2
- new net N$10: R9.2, U$1.AC1, X1-1.KL, X2-1.KL, X3-1.KL
- new net N$19: R4.2, U$4.CH_PD
- net 5V: now also R8.2
- net ESP8266_TX: now also B1.15(RX3), U$4.TXD; no longer ESP8266-RIGHT.1
- net GND0: no longer DHT.2, LDR.2, TMP1.2, TMP2.2
- net GND1: now also C1.-, CX1.2, JP1.4, U$4.GND; no longer ESP8266-RIGHT.8, RELAY_1.2, RELAY_2.2
- net N$2: now also R9.1
- net N$8: now also U$4.RXD; no longer ESP8266-RIGHT.2
- net POWER_SUPPLY_3.3V: now also C1.+, U$4.VCC; no longer ESP8266-LEFT.8
- net POWER_SUPPLY_5V: now also CX1.1, JP1.1, S1.1; no longer RELAY_1.3, RELAY_2.3, U$1.DC+
- net RELAY_1: now also B1.A1(TX0), JP1.2; no longer RELAY_1.1
- net RELAY_2: now also B1.A0(RX0), JP1.3; no longer RELAY_2.1
- net TMP: now also R8.1
Other:
- moved on the sheet: DHT, LDR, R4, R5, R6, R7, TMP1, TMP2
